Commit message: gecko updated

File: gecko/gecko_description/urdf/camera.xacro (robot description, xacro)
@@ -25,6 +25,6 @@
     <joint name="camera_joint" type="fixed">
     <axis xyz="0 0 0" />
-    <origin xyz="0 0.3 0.2" rpy="0 ${pi/2} ${-pi/2}"/>
-    <parent link="base_link"/>
+    <origin xyz="0.03 0 0.13" rpy="0 0.28 0"/>
+    <parent link="hokuyo_link"/>
     <child link="camera_link"/>
   </joint>

File: gecko/gecko_description/urdf/gecko.xacro (robot description, xacro)
@@ -339,5 +339,5 @@
     <origin xyz="0 0.15 0"/>
     </joint>
-    <!-- /////////////// 4+4 tires ///////////////////////////////////////-->
+    <!-- /////////////// 4x4 tires ///////////////////////////////////////-->
 <link name="upper_left_cylinder">
     <xacro:tire/>
@@ -412,4 +412,95 @@
     <origin xyz="-0.6 0 0"/>
     </joint>
+<!--////////////////////////// fixed bar ////////////////////////////////////////////////-->
+ <link name="left_inside_leg">
+    <visual>
+      <geometry>
+        <box size="0.03 1 0.03"/>
+      </geometry>
+      <origin rpy="0 0 0" xyz="0 0 0"/>
+      <material name="white"/>
+    </visual>
+    <collision>
+    <geometry>
+        <box size="0.03 1 0.03"/>
+      </geometry>
+      <origin rpy="0 0 0" xyz="0 0 0"/>
+      <material name="red"/>
+      </collision>
+    <xacro:default_low_inertial />
+  </link>
+  <joint name="left_inside_leg_joint" type="fixed">
+    <parent link="base_link"/>
+    <child link="left_inside_leg"/>
+    <origin xyz="0.24 0.05 0.2"/>
+    </joint>
+     <link name="right_inside_leg">
+    <visual>
+      <geometry>
+        <box size="0.03 1 0.03"/>
+      </geometry>
+      <origin rpy="0 0 0" xyz="0 0 0"/>
+      <material name="white"/>
+    </visual>
+    <collision>
+    <geometry>
+        <box size="0.03 1 0.03"/>
+      </geometry>
+      <origin rpy="0 0 0" xyz="0 0 0"/>
+      <material name="red"/>
+      </collision>
+    <xacro:default_low_inertial />
+  </link>
+  <joint name="right_inside_leg_joint" type="fixed">
+    <parent link="base_link"/>
+    <child link="right_inside_leg"/>
+    <origin xyz="-0.24 0.05 0.2"/>
+    </joint>
+<link name="upper_inside_leg">
+    <visual>
+      <geometry>
+        <box size="0.445 0.03 0.03"/>
+      </geometry>
+      <origin rpy="0 0 0" xyz="0 0 0"/>
+      <material name="white"/>
+    </visual>
+    <collision>
+    <geometry>
+       <box size="0.445 0.03 0.03"/>
+      </geometry>
+      <origin rpy="0 0 0" xyz="0 0 0"/>
+      <material name="red"/>
+          </collision>
+    <xacro:default_low_inertial />
+  </link>
+  <joint name="upper_inside_leg_joint" type="fixed">
+    <parent link="base_link"/>
+    <child link="upper_inside_leg"/>
+    <axis xyz="1 0 0"/>
+    <origin xyz="0 -0.435 0.2"/>
+  </joint>
+  <link name="lower_inside_leg">
+    <visual>
+      <geometry>
+        <box size="0.445 0.03 0.03"/>
+      </geometry>
+      <origin rpy="0 0 0" xyz="0 0 0"/>
+      <material name="white"/>
+    </visual>
+    <collision>
+    <geometry>
+       <box size="0.445 0.03 0.03"/>
+      </geometry>
+      <origin rpy="0 0 0" xyz="0 0 0"/>
+      <material name="red"/>
+          </collision>
+    <xacro:default_low_inertial />
+  </link>
+  <joint name="lower_inside_leg_joint" type="fixed">
+    <parent link="base_link"/>
+    <child link="lower_inside_leg"/>
+    <axis xyz="1 0 0"/>
+    <origin xyz="0 0.538 0.2"/>
+  </joint>
 <!-- /////////////// transmissions ///////////////////////////////////////-->
 <transmission name="tran_upper_left_bar_1_joint">
@@ -453,3 +544,23 @@
     </actuator>
   </transmission>
+  <transmission name="tran_horizontal_traslation_link_joint">
+    <type>transmission_interface/SimpleTransmission</type>
+    <joint name="horizontal_traslation_link_joint">
+      <hardwareInterface>hardware_interface/PositionJointInterface</hardwareInterface>
+    </joint>
+    <actuator name="motor_horizontal_traslation_link_joint">
+      <hardwareInterface>hardware_interface/PositionJointInterface</hardwareInterface>
+      <mechanicalReduction>1</mechanicalReduction>
+    </actuator>
+  </transmission>
+   <transmission name="tran_hokuyo_joint">
+    <type>transmission_interface/SimpleTransmission</type>
+    <joint name="hokuyo_joint">
+      <hardwareInterface>hardware_interface/PositionJointInterface</hardwareInterface>
+    </joint>
+    <actuator name="motor_hokuyo_joint">
+      <hardwareInterface>hardware_interface/PositionJointInterface</hardwareInterface>
+      <mechanicalReduction>1</mechanicalReduction>
+    </actuator>
+  </transmission>
 </robot>

File: gecko/gecko_description/urdf/laser.xacro (robot description, xacro)
@@ -17,14 +17,43 @@
     </visual>
     <inertial>
-      <mass value="1e-5" />
+      <mass value="1" />
       <origin xyz="0 0 0" rpy="0 0 0"/>
-      <inertia ixx="1e-6" ixy="0" ixz="0" iyy="1e-6" iyz="0" izz="1e-6" />
+      <inertia ixx="1" ixy="0" ixz="0" iyy="1" iyz="0" izz="1" />
     </inertial>
   </link>
-   <joint name="hokuyo_joint" type="fixed">
+   <joint name="hokuyo_joint" type="prismatic">
     <axis xyz="0 1 0" />
-    <origin xyz="0 0.4 0.2" rpy="0 1.3 ${-pi/2}"/>
+    <origin xyz="0 0 0" rpy="0 1.3 ${-pi/2}"/>
+    <parent link="horizontal_traslation_link"/>
+    <child link="hokuyo_link"/>
+    <limit effort="10.0" lower="-0.2" upper="0.2" velocity="0.5"/>
+  </joint>
+  <link name="horizontal_traslation_link">
+      <visual>
+      <origin xyz="0 0 0" rpy="0 0 0"/>
+	<geometry>
+    <box size="0.01 0.01 0.01"/>
+      </geometry>
+    </visual>
+    <collision>
+      <origin xyz="0 0 0" rpy="0 0 0"/>
+      <geometry>
+    <box size="0 0 0"/>
+      </geometry>
+    </collision>
+    <inertial>
+      <mass value="0.5" />
+      <origin xyz="0 0 0" rpy="0 0 0"/>
+                <inertia ixx="1.0" ixy="0.0" ixz="0.0"
+                     iyy="1.0" iyz="0.0"
+                     izz="1.0" />
+    </inertial>
+  </link>
+   <joint name="horizontal_traslation_link_joint" type="prismatic">
+    <axis xyz="0 1 0" />
+    <origin xyz="0 0.4 0.2" rpy="0 0 0"/>
     <parent link="base_link"/>
-    <child link="hokuyo_link"/>
+    <child link="horizontal_traslation_link"/>
+    <limit effort="1000" lower="-0.66" upper="0.08" velocity="0.5"/>
   </joint>
    <!-- hokuyo -->
@@ -50,8 +79,4 @@
         <noise>
           <type>gaussian</type>
-          <!-- Noise parameters based on published spec for Hokuyo laser
-               achieving "+-30mm" accuracy at range < 10m.  A mean of 0.0m and
-               stddev of 0.01m will put 99.7% of samples within 0.03m of the true
-               reading. -->
           <mean>0.0</mean>
           <stddev>0.01</stddev>
